File: HB-RC-6-PBU-LED.kicad_pcb (KiCad board)
At the start: 2 copper layers, 50 x 50 mm, 34 parts, among them IC1 CC1101, J2 ISP, J3 FTDI, SW1 Config, SW2 BTN1, SW3 BTN2, SW4 BTN3, SW5 BTN4, SW6 BTN5, SW7 BTN6, U1 ATmega644A-AU, U3 SN74LVC1T45DBV

Commit message: Add files via upload
Parts:
- removed the C4 at (195.7, 59.0)
- removed the C5 at (204.0, 68.5)
- added C10: 100n, Capacitor_SMD:C_0805_2012Metric_Pad1.18x1.45mm_HandSolder, F.Cu at (204.0, 68.5)
- added C9: 100n, Capacitor_SMD:C_0805_2012Metric_Pad1.18x1.45mm_HandSolder, F.Cu at (195.8, 59.0)
- added D10: WS2812-2020, WS2812-2020:LED_WS2812-2020, F.Cu at (178.0, 75.0)
- added D11: WS2812-2020, WS2812-2020:LED_WS2812-2020, F.Cu at (178.0, 93.0)
- added D12: WS2812-2020, WS2812-2020:LED_WS2812-2020, F.Cu at (212.0, 57.0)
- added D13: WS2812-2020, WS2812-2020:LED_WS2812-2020, F.Cu at (212.0, 75.0)
- added D14: WS2812-2020, WS2812-2020:LED_WS2812-2020, F.Cu at (212.0, 93.0)
- added D9: WS2812-2020, WS2812-2020:LED_WS2812-2020, F.Cu at (178.0, 57.0)
- added J1: Maincon, Connector_PinHeader_2.54mm:PinHeader_2x04_P2.54mm_Vertical_SMD, B.Cu at (194.7, 74.8)
- added Q1: IRLML9301, Package_TO_SOT_SMD:SOT-23, F.Cu at (188.0, 56.8)
- added R5: 1K, Resistor_SMD:R_0805_2012Metric_Pad1.20x1.40mm_HandSolder, F.Cu at (199.0, 59.0)
- added R6: 100K, Resistor_SMD:R_0805_2012Metric_Pad1.20x1.40mm_HandSolder, F.Cu at (188.0, 59.8)
- renumbered C2 to C1, C7 to C2, C8 to C3, C9 to C4, C10 to C5, C11 to C6, C12 to C7, C13 to C8
Connections:
- C3 pad 2: +5V -> /WS2812B_VCC
- C4 pad 2: +5V -> /WS2812B_VCC
- C5 pad 2: +5V -> /WS2812B_VCC
- C6 pad 2: +5V -> /WS2812B_VCC
- C7 pad 2: +5V -> /WS2812B_VCC
- C8 pad 2: +5V -> /WS2812B_VCC
- D3 pad 4: +5V -> /WS2812B_VCC
- D4 pad 4: +5V -> /WS2812B_VCC
- D5 pad 4: +5V -> /WS2812B_VCC
- D6 pad 4: +5V -> /WS2812B_VCC
- D7 pad 4: +5V -> /WS2812B_VCC
- D8 pad 4: +5V -> /WS2812B_VCC
- U1 pad 23: Net-(U1-Pad23) -> /WS2812B_IO
Routing:
- net /WS2812B_VCC: track 0.00 -> 125.4 mm
- net +5V: track 119.6 -> 36.9 mm, vias 0 -> 1
- net Net-(Q1-Pad1): track 0.00 -> 15.6 mm
- net /TX: track 24.6 -> 35.7 mm
- net /RX: track 27.7 -> 38.0 mm
- net +3V3: track 126.5 -> 135.1 mm, vias 2 -> 5
- net GND: track 78.0 -> 74.4 mm, vias 8 -> 32
- net /WS2812B_IO: track 0.00 -> 2.31 mm
- net Net-(D12-Pad1): track 15.2 -> 17.2 mm
- net Net-(D11-Pad1): track 80.5 -> 82.5 mm
- net Net-(D10-Pad3): track 15.2 -> 17.2 mm
- net Net-(D13-Pad1): track 15.2 -> 17.1 mm
- net Net-(D10-Pad1): track 15.2 -> 17.1 mm
- net /WS2812B_LED_3V3_Lvl: track 24.9 -> 23.3 mm
- net /WS2812B_LED_5V_Lvl: track 4.79 -> 5.77 mm
Other:
- board text added: "3V3"
- board text added: "DTR"
- board text added: "GND"
- board text added: "MISO"
- board text added: "MOSI"
- board text added: "RESET"
- board text added: "RX"
- board text added: "SCK"
- board text added: "TX"
- board text added: "°"

Commit message: Bugfix
Parts:
- R1, R2: value 330 -> 240
- turned U3 to 180 degrees
- renumbered IC1 to U2
Connections:
- J3 pad 2: /TX -> /RX
- J3 pad 3: /RX -> /TX
- U3 pad 3: /WS2812B_LED_5V_Lvl -> /WS2812B_LED_3V3_Lvl
- U3 pad 4: /WS2812B_LED_3V3_Lvl -> /WS2812B_LED_5V_Lvl
Routing:
- net GND: track 74.4 -> 69.8 mm, vias 32 -> 36
- net /WS2812B_LED_3V3_Lvl: track 23.3 -> 27.9 mm
- net /TX: track 35.7 -> 39.2 mm
- net /RX: track 38.0 -> 35.4 mm
- net +3V3: track 135.1 -> 134.3 mm
- net /BTN6: track 38.9 -> 39.7 mm, vias 4 -> 2
- net +5V: track 36.9 -> 36.2 mm
- net /WS2812B_LED_5V_Lvl: track 5.77 -> 5.26 mm
